File: led matrix.kicad_sch (KiCad schematic)
At the start: 10 parts, among them J41 Conn_01x03_MountingPin, J42 Conn_01x03_MountingPin, U40 LP5814DRLR

Commit message: outline
Parts:
- removed C40, C5: 10uF, Capacitor_SMD:C_0805_2012Metric, symbol Device:C
- removed C55: 1uF, Capacitor_SMD:C_0603_1608Metric, symbol Device:C
- removed D36, D37, D38, D39: LED, PCM_LED_SMD_AKL:LED_PLCC_2835, symbol Device:LED
- removed J41, J42: Conn_01x03_MountingPin, Connector_JST:JST_SH_SM03B-SRSS-TB_1x03-1MP_P1.00mm_Horizontal, symbol Connector_Generic_MountingPin:Conn_01x03_MountingPin
- removed U40: LP5814DRLR, Package_TO_SOT_SMD:SOT-583-8, symbol gachlilit:LP5814DRLR
Other:
- note removed: "argb in"
- note removed: "argb out"
- note removed: "blacklight"
- note removed: "rgb power in"
